Commit message: Add drive wheels with continuous joints

File: merobot_description/urdf/merobot.urdf.xacro (robot description, xacro)
@@ -6,7 +6,17 @@
   <xacro:property name="base_height" value="0.1"/>
   <xacro:property name="base_mass" value="2.0"/>
-    <material name="gray">
+  <!-- Wheel dimensions -->
+  <xacro:property name="wheel_radius" value="0.06"/>
+  <xacro:property name="wheel_width" value="0.04"/>
+  <xacro:property name="wheel_mass" value="0.3"/>
+  <xacro:property name="wheel_x_offset" value="0.05"/>
+  <!-- Colors -->
+  <material name="gray">
     <color rgba="0.6 0.6 0.6 1.0"/>
   </material>
+  <material name="black">
+    <color rgba="0.1 0.1 0.1 1.0"/>
+  </material>
+  <!-- Chassis -->
   <link name="base_link">
     <visual>
@@ -30,9 +40,46 @@
     </inertial>
   </link>
+  <!-- Ground reference point -->
   <link name="base_footprint"/>
   <joint name="base_footprint_joint" type="fixed">
     <parent link="base_footprint"/>
     <child link="base_link"/>
-    <origin xyz="0 0 ${base_height/2}" rpy="0 0 0"/>
+    <origin xyz="0 0 ${wheel_radius}" rpy="0 0 0"/>
   </joint>
+  <!-- Wheel macro: write once, use twice -->
+  <xacro:macro name="wheel" params="prefix y_reflect">
+    <link name="${prefix}_wheel">
+      <visual>
+        <origin xyz="0 0 0" rpy="${pi/2} 0 0"/>
+        <geometry>
+          <cylinder radius="${wheel_radius}" length="${wheel_width}"/>
+        </geometry>
+        <material name="black"/>
+      </visual>
+      <collision>
+        <origin xyz="0 0 0" rpy="${pi/2} 0 0"/>
+        <geometry>
+          <cylinder radius="${wheel_radius}" length="${wheel_width}"/>
+        </geometry>
+      </collision>
+      <inertial>
+        <origin xyz="0 0 0" rpy="${pi/2} 0 0"/>
+        <mass value="${wheel_mass}"/>
+        <inertia
+          ixx="${wheel_mass/12.0*(3*wheel_radius*wheel_radius + wheel_width*wheel_width)}"
+          iyy="${wheel_mass/12.0*(3*wheel_radius*wheel_radius + wheel_width*wheel_width)}"
+          izz="${wheel_mass/2.0*wheel_radius*wheel_radius}"
+          ixy="0" ixz="0" iyz="0"/>
+      </inertial>
+    </link>
+    <joint name="${prefix}_wheel_joint" type="continuous">
+      <parent link="base_link"/>
+      <child link="${prefix}_wheel"/>
+      <origin xyz="${wheel_x_offset} ${y_reflect*(base_width/2 + wheel_width/2)} 0" rpy="0 0 0"/>
+      <axis xyz="0 1 0"/>
+    </joint>
+  </xacro:macro>
+  <!-- Use the macro twice -->
+  <xacro:wheel prefix="left" y_reflect="1"/>
+  <xacro:wheel prefix="right" y_reflect="-1"/>
 </robot>

Commit message: Add caster wheel and complete robot base

File: merobot_description/urdf/merobot.urdf.xacro (robot description, xacro)
@@ -11,4 +11,8 @@
   <xacro:property name="wheel_mass" value="0.3"/>
   <xacro:property name="wheel_x_offset" value="0.05"/>
+  <!-- Caster dimensions -->
+  <xacro:property name="caster_radius" value="0.02"/>
+  <xacro:property name="caster_mass" value="0.05"/>
+  <xacro:property name="caster_x_offset" value="-0.11"/>
   <!-- Colors -->
   <material name="gray">
@@ -83,3 +87,30 @@
   <xacro:wheel prefix="left" y_reflect="1"/>
   <xacro:wheel prefix="right" y_reflect="-1"/>
+  <!-- Caster wheel (free-rolling ball at the back) -->
+  <link name="caster_wheel">
+    <visual>
+      <geometry>
+        <sphere radius="${caster_radius}"/>
+      </geometry>
+      <material name="black"/>
+    </visual>
+    <collision>
+      <geometry>
+        <sphere radius="${caster_radius}"/>
+      </geometry>
+    </collision>
+    <inertial>
+      <mass value="${caster_mass}"/>
+      <inertia
+        ixx="${2.0/5.0*caster_mass*caster_radius*caster_radius}"
+        iyy="${2.0/5.0*caster_mass*caster_radius*caster_radius}"
+        izz="${2.0/5.0*caster_mass*caster_radius*caster_radius}"
+        ixy="0" ixz="0" iyz="0"/>
+    </inertial>
+  </link>
+  <joint name="caster_wheel_joint" type="fixed">
+    <parent link="base_link"/>
+    <child link="caster_wheel"/>
+    <origin xyz="${caster_x_offset} 0 ${-(wheel_radius - caster_radius)}" rpy="0 0 0"/>
+  </joint>
 </robot>

Commit message: Add lidar sensor, obstacle world and RViz in simulation

File: merobot_description/urdf/merobot.urdf.xacro (robot description, xacro)
@@ -1,19 +1,24 @@
 <?xml version="1.0"?>
 <robot name="merobot" xmlns:xacro="http://www.ros.org/wiki/xacro">
-  <!-- Chassis dimensions (meters, kilograms) -->
+  <!-- ==================== Dimensions ==================== -->
+  <!-- Chassis (meters, kilograms) -->
   <xacro:property name="base_length" value="0.3"/>
   <xacro:property name="base_width" value="0.3"/>
   <xacro:property name="base_height" value="0.1"/>
   <xacro:property name="base_mass" value="2.0"/>
-  <!-- Wheel dimensions -->
+  <!-- Wheels -->
   <xacro:property name="wheel_radius" value="0.06"/>
   <xacro:property name="wheel_width" value="0.04"/>
   <xacro:property name="wheel_mass" value="0.3"/>
   <xacro:property name="wheel_x_offset" value="0.05"/>
-  <!-- Caster dimensions -->
+  <!-- Caster -->
   <xacro:property name="caster_radius" value="0.02"/>
   <xacro:property name="caster_mass" value="0.05"/>
   <xacro:property name="caster_x_offset" value="-0.11"/>
-  <!-- Colors -->
+  <!-- Lidar -->
+  <xacro:property name="lidar_radius" value="0.05"/>
+  <xacro:property name="lidar_height" value="0.04"/>
+  <xacro:property name="lidar_mass" value="0.1"/>
+  <!-- ==================== Colors ==================== -->
   <material name="gray">
     <color rgba="0.6 0.6 0.6 1.0"/>
@@ -22,5 +27,8 @@
     <color rgba="0.1 0.1 0.1 1.0"/>
   </material>
-  <!-- Chassis -->
+  <material name="red">
+    <color rgba="0.8 0.1 0.1 1.0"/>
+  </material>
+  <!-- ==================== Chassis ==================== -->
   <link name="base_link">
     <visual>
@@ -51,5 +59,5 @@
     <origin xyz="0 0 ${wheel_radius}" rpy="0 0 0"/>
   </joint>
-  <!-- Wheel macro: write once, use twice -->
+  <!-- ==================== Wheels ==================== -->
   <xacro:macro name="wheel" params="prefix y_reflect">
     <link name="${prefix}_wheel">
@@ -84,8 +92,7 @@
     </joint>
   </xacro:macro>
-  <!-- Use the macro twice -->
   <xacro:wheel prefix="left" y_reflect="1"/>
   <xacro:wheel prefix="right" y_reflect="-1"/>
-  <!-- Caster wheel (free-rolling ball at the back) -->
+  <!-- ==================== Caster ==================== -->
   <link name="caster_wheel">
     <visual>
@@ -114,5 +121,32 @@
     <origin xyz="${caster_x_offset} 0 ${-(wheel_radius - caster_radius)}" rpy="0 0 0"/>
   </joint>
-    <!-- ==================== Gazebo ==================== -->
+  <!-- ==================== Lidar ==================== -->
+  <link name="lidar_link">
+    <visual>
+      <geometry>
+        <cylinder radius="${lidar_radius}" length="${lidar_height}"/>
+      </geometry>
+      <material name="red"/>
+    </visual>
+    <collision>
+      <geometry>
+        <cylinder radius="${lidar_radius}" length="${lidar_height}"/>
+      </geometry>
+    </collision>
+    <inertial>
+      <mass value="${lidar_mass}"/>
+      <inertia
+        ixx="${lidar_mass/12.0*(3*lidar_radius*lidar_radius + lidar_height*lidar_height)}"
+        iyy="${lidar_mass/12.0*(3*lidar_radius*lidar_radius + lidar_height*lidar_height)}"
+        izz="${lidar_mass/2.0*lidar_radius*lidar_radius}"
+        ixy="0" ixz="0" iyz="0"/>
+    </inertial>
+  </link>
+  <joint name="lidar_joint" type="fixed">
+    <parent link="base_link"/>
+    <child link="lidar_link"/>
+    <origin xyz="0 0 ${base_height/2 + lidar_height/2}" rpy="0 0 0"/>
+  </joint>
+  <!-- ==================== Gazebo ==================== -->
   <gazebo>
     <!-- Motors: turns velocity commands into wheel rotation -->
@@ -137,5 +171,30 @@
   <gazebo reference="caster_wheel">
     <mu1>0.0</mu1>
-    <mu2>0.0</mu2>
+    <mu2>0.0</mu2>    <mu2>0.0</mu2>
+  </gazebo>
+  <!-- Lidar sensor -->
+  <gazebo reference="lidar_link">
+    <sensor name="lidar" type="gpu_lidar">
+      <topic>scan</topic>
+      <gz_frame_id>lidar_link</gz_frame_id>
+      <update_rate>10</update_rate>
+      <always_on>true</always_on>
+      <visualize>true</visualize>
+      <lidar>
+        <scan>
+          <horizontal>
+            <samples>360</samples>
+            <resolution>1</resolution>
+            <min_angle>-3.14159</min_angle>
+            <max_angle>3.14159</max_angle>
+          </horizontal>
+        </scan>
+        <range>
+          <min>0.12</min>
+          <max>8.0</max>
+          <resolution>0.01</resolution>
+        </range>
+      </lidar>
+    </sensor>
   </gazebo>
 </robot>
